Commit message: Update project

File: description/ros2_control.xacro (robot description, xacro)
@@ -6,6 +6,4 @@
             <param name="left_wheel_name">base_left_wheel_joint</param>
             <param name="right_wheel_name">base_right_wheel_joint</param>
-            <param name="rright_wheel_name">base_right_wheel2_joint</param>
-            <param name="rleft_wheel_name">base_left_wheel2_joint</param>
             <param name="loop_rate">30</param>
             <param name="device">/dev/ttyACM0</param>
@@ -26,21 +24,5 @@
             <state_interface name="velocity"/>
         </joint>
-        <joint name="base_left_wheel2_joint">
-            <command_interface name="velocity">
-                <param name="min">-10</param>
-                <param name="max">10</param>
-            </command_interface>
-            <state_interface name="position"/>
-            <state_interface name="velocity"/>
-        </joint>
         <joint name="base_right_wheel_joint">
-            <command_interface name="velocity">
-                <param name="min">-10</param>
-                <param name="max">10</param>
-            </command_interface>
-            <state_interface name="position"/>
-            <state_interface name="velocity"/>
-        </joint>
-        <joint name="base_right_wheel2_joint">
             <command_interface name="velocity">
                 <param name="min">-10</param>
